Commit message: Hell yeah

File: painting_cell/urdf/painting_cell.urdf (robot description, URDF)
Before this commit: robot painting_cell, 18 links, 17 joints
Links:
- removed link world
- link painting_cell: geometry collision mesh filename=package://painting_cell/meshes/cell.STL; visual mesh filename=package://painting_cell/meshes/cell.STL
Joints:
- removed joint fixed_link_to_world

Commit message: gazebo simulation works now

File: painting_cell/urdf/painting_cell.urdf (robot description, URDF)
Before this commit: robot painting_cell, 17 links, 16 joints
Joints:
- joint foundation: origin xyz=0 0 0 rpy=0 0 1.5708 -> xyz=0 0 0 rpy=0 0 0
- joint joint_0_simon: limit lower=0 upper=0 effort=0 velocity=0 -> (none)
- joint joint_1_flo: limit lower=-3.1416 upper=3.1416 effort=0 velocity=0 -> lower=-3.1416 upper=3.1416 effort=5 velocity=0
- joint joint_1_simon: limit lower=-3.1416 upper=3.1416 effort=0 velocity=0 -> lower=-3.1416 upper=3.1416 effort=5 velocity=0
- joint joint_2_flo: limit lower=-3.1416 upper=3.1416 effort=0 velocity=0 -> lower=-3.1416 upper=3.1416 effort=5 velocity=0
- joint joint_2_simon: limit lower=-3.1416 upper=3.1416 effort=0 velocity=0 -> lower=-3.1416 upper=3.1416 effort=5 velocity=0
- joint joint_3_flo: limit lower=-3.1416 upper=3.1416 effort=0 velocity=0 -> lower=-3.1416 upper=3.1416 effort=5 velocity=0
- joint joint_3_simon: limit lower=-3.1416 upper=3.1416 effort=0 velocity=0 -> lower=-3.1416 upper=3.1416 effort=5 velocity=0
- joint joint_4_flo: limit lower=-3.1416 upper=3.1416 effort=0 velocity=0 -> lower=-3.1416 upper=3.1416 effort=5 velocity=0
- joint joint_4_simon: limit lower=-3.1416 upper=3.1416 effort=0 velocity=0 -> lower=-3.1416 upper=3.1416 effort=5 velocity=0
- joint joint_5_flo: limit lower=-3.1416 upper=3.1416 effort=0 velocity=0 -> lower=-3.1416 upper=3.1416 effort=5 velocity=0
- joint joint_5_simon: limit lower=-3.1416 upper=3.1416 effort=0 velocity=0 -> lower=-3.1416 upper=3.1416 effort=5 velocity=0
- joint joint_6_flo: limit lower=-3.1416 upper=3.1416 effort=0 velocity=0 -> lower=-3.1416 upper=3.1416 effort=5 velocity=0
- joint joint_6_simon: limit lower=-3.1416 upper=3.1416 effort=0 velocity=0 -> lower=-3.1416 upper=3.1416 effort=5 velocity=0
- joint joint_turn_table: limit lower=-3.1416 upper=3.1416 effort=0 velocity=3.1416 -> lower=-3.1416 upper=3.1416 effort=5 velocity=3.1416

Commit message: Gazebo sim startet und lässt bewegungen aus moveit zu

File: painting_cell/urdf/painting_cell.urdf (robot description, URDF)
Before this commit: robot painting_cell, 17 links, 16 joints
Joints:
- joint joint_1_flo: limit lower=-3.1416 upper=3.1416 effort=5 velocity=0 -> lower=-3.1416 upper=3.1416 effort=10 velocity=3.1416
- joint joint_1_simon: limit lower=-3.1416 upper=3.1416 effort=5 velocity=0 -> lower=-3.1416 upper=3.1416 effort=10 velocity=3.1416
- joint joint_2_flo: limit lower=-3.1416 upper=3.1416 effort=5 velocity=0 -> lower=-3.1416 upper=3.1416 effort=10 velocity=3.1416
- joint joint_2_simon: limit lower=-3.1416 upper=3.1416 effort=5 velocity=0 -> lower=-3.1416 upper=3.1416 effort=10 velocity=3.1416
- joint joint_3_flo: limit lower=-3.1416 upper=3.1416 effort=5 velocity=0 -> lower=-3.1416 upper=3.1416 effort=10 velocity=3.1416
- joint joint_3_simon: limit lower=-3.1416 upper=3.1416 effort=5 velocity=0 -> lower=-3.1416 upper=3.1416 effort=10 velocity=3.1416
- joint joint_4_flo: limit lower=-3.1416 upper=3.1416 effort=5 velocity=0 -> lower=-3.1416 upper=3.1416 effort=10 velocity=6.2832
- joint joint_4_simon: limit lower=-3.1416 upper=3.1416 effort=5 velocity=0 -> lower=-3.1416 upper=3.1416 effort=10 velocity=6.2832
- joint joint_5_flo: limit lower=-3.1416 upper=3.1416 effort=5 velocity=0 -> lower=-3.1416 upper=3.1416 effort=10 velocity=6.2832
- joint joint_5_simon: limit lower=-3.1416 upper=3.1416 effort=5 velocity=0 -> lower=-3.1416 upper=3.1416 effort=10 velocity=6.2832
- joint joint_6_flo: limit lower=-3.1416 upper=3.1416 effort=5 velocity=0 -> lower=-3.1416 upper=3.1416 effort=10 velocity=6.2832
- joint joint_6_simon: limit lower=-3.1416 upper=3.1416 effort=5 velocity=0 -> lower=-3.1416 upper=3.1416 effort=10 velocity=6.2832
- joint joint_turn_table: limit lower=-3.1416 upper=3.1416 effort=5 velocity=3.1416 -> lower=-3.1416 upper=3.1416 effort=10 velocity=3.1416

Commit message: jpint limit for turn table, and turntable points

File: painting_cell/urdf/painting_cell.urdf (robot description, URDF)
Before this commit: robot painting_cell, 17 links, 16 joints
Joints:
- joint joint_turn_table: limit lower=-3.1416 upper=3.1416 effort=10 velocity=3.1416 -> lower=-1000 upper=1000 effort=10 velocity=6.1832

Commit message: addded knights and fixed gazebo jumping

File: painting_cell/urdf/painting_cell.urdf (robot description, URDF)
Before this commit: robot painting_cell, 17 links, 16 joints
Links:
- added link knight_1, mass 0.809118720487137; collision mesh filename=package://painting_cell/meshes/knight_1.STL; visual mesh filename=package://painting_cell/meshes/knight_1.STL
- added link knight_2, mass 0.809113158889413; collision mesh filename=package://painting_cell/meshes/knight_2.STL; visual mesh filename=package://painting_cell/meshes/knight_2.STL
- added link knight_3, mass 0.809122251382701; collision mesh filename=package://painting_cell/meshes/knight_3.STL; visual mesh filename=package://painting_cell/meshes/knight_3.STL
- added link world
Joints:
- added joint fixed_link_to_world: type fixed, parent world, child a_foundation
- added joint joint_knight_1: type fixed, parent turn_table, child knight_1, origin xyz=-0.0065718 0.025 0.58785 rpy=1.5708 1.5707 0, axis 1 0 0, limit lower=0 upper=0 effort=0 velocity=0
- added joint joint_knight_2: type fixed, parent turn_table, child knight_2, origin xyz=0.55143 0.025 -0.31078 rpy=1.5708 -0.52348 3.1416, axis 0 0 0
- added joint joint_knight_3: type fixed, parent turn_table, child knight_3, origin xyz=-0.54486 0.025 -0.32217 rpy=-1.5708 -0.52372 0, axis 0 0 0
- joint joint_turn_table: limit lower=-1000 upper=1000 effort=10 velocity=6.1832 -> lower=-6.2833 upper=6.2833 effort=10 velocity=6.1832

Commit message: cure process works simulated

File: painting_cell/urdf/painting_cell.urdf (robot description, URDF)
Before this commit: robot painting_cell, 21 links, 20 joints
Links:
- removed link knight_2
- removed link knight_3
Joints:
- removed joint joint_knight_2
- removed joint joint_knight_3

Commit message: simon dont work

File: painting_cell/urdf/painting_cell.urdf (robot description, URDF)
Before this commit: robot painting_cell, 19 links, 18 joints
Joints:
- joint joint_6_flo: limit lower=-3.1416 upper=3.1416 effort=10 velocity=6.2832 -> lower=-6.2832 upper=6.2832 effort=10 velocity=6.2832
- joint joint_6_simon: limit lower=-3.1416 upper=3.1416 effort=10 velocity=6.2832 -> lower=-6.2832 upper=6.2832 effort=10 velocity=6.2832

Commit message: changed turn_table to continuous joint

File: painting_cell/urdf/painting_cell.urdf (robot description, URDF)
Before this commit: robot painting_cell, 19 links, 18 joints
Joints:
- joint joint_turn_table: limit lower=-6.2833 upper=6.2833 effort=10 velocity=6.1832 -> effort=10 velocity=6.1832; type revolute -> continuous

Commit message: error solved,  it was the effort limit

File: painting_cell/urdf/painting_cell.urdf (robot description, URDF)
Before this commit: robot painting_cell, 19 links, 18 joints
Joints:
- joint joint_1_flo: limit lower=-3.1416 upper=3.1416 effort=10 velocity=3.1416 -> lower=-3.1416 upper=3.1416 effort=10000 velocity=3.1416
- joint joint_1_simon: limit lower=-3.1416 upper=3.1416 effort=10 velocity=3.1416 -> lower=-3.1416 upper=3.1416 effort=10000 velocity=3.1416
- joint joint_2_flo: limit lower=-3.1416 upper=3.1416 effort=10 velocity=3.1416 -> lower=-3.1416 upper=3.1416 effort=10000 velocity=3.1416
- joint joint_2_simon: limit lower=-3.1416 upper=3.1416 effort=10 velocity=3.1416 -> lower=-3.1416 upper=3.1416 effort=10000 velocity=3.1416
- joint joint_3_flo: limit lower=-3.1416 upper=3.1416 effort=10 velocity=3.1416 -> lower=-3.1416 upper=3.1416 effort=10000 velocity=3.1416
- joint joint_3_simon: limit lower=-3.1416 upper=3.1416 effort=10 velocity=3.1416 -> lower=-3.1416 upper=3.1416 effort=10000 velocity=3.1416
- joint joint_4_flo: limit lower=-3.1416 upper=3.1416 effort=10 velocity=6.2832 -> lower=-3.1416 upper=3.1416 effort=10000 velocity=6.2832
- joint joint_4_simon: limit lower=-3.1416 upper=3.1416 effort=10 velocity=6.2832 -> lower=-3.1416 upper=3.1416 effort=10000 velocity=6.2832
- joint joint_5_flo: limit lower=-3.1416 upper=3.1416 effort=10 velocity=6.2832 -> lower=-3.1416 upper=3.1416 effort=10000 velocity=6.2832
- joint joint_5_simon: limit lower=-3.1416 upper=3.1416 effort=10 velocity=6.2832 -> lower=-3.1416 upper=3.1416 effort=10000 velocity=6.2832
- joint joint_6_flo: limit lower=-6.2832 upper=6.2832 effort=10 velocity=6.2832 -> lower=-6.2832 upper=6.2832 effort=10000 velocity=6.2832
- joint joint_6_simon: limit lower=-6.2832 upper=6.2832 effort=10 velocity=6.2832 -> lower=-6.2832 upper=6.2832 effort=10000 velocity=6.2832
- joint joint_turn_table: limit effort=10 velocity=6.1832 -> effort=10000 velocity=6.1832

Commit message: TCP Movement works, it was the tuples

File: painting_cell/urdf/painting_cell.urdf (robot description, URDF)
Before this commit: robot painting_cell, 19 links, 18 joints
Joints:
- joint joint_1_flo: limit lower=-3.1416 upper=3.1416 effort=10000 velocity=3.1416 -> lower=-3.1416 upper=3.1416 effort=10 velocity=3.1416
- joint joint_2_flo: limit lower=-3.1416 upper=3.1416 effort=10000 velocity=3.1416 -> lower=-3.1416 upper=3.1416 effort=10 velocity=3.1416
- joint joint_3_flo: limit lower=-3.1416 upper=3.1416 effort=10000 velocity=3.1416 -> lower=-3.1416 upper=3.1416 effort=10 velocity=3.1416
- joint joint_4_flo: limit lower=-3.1416 upper=3.1416 effort=10000 velocity=6.2832 -> lower=-3.1416 upper=3.1416 effort=10 velocity=6.2832
- joint joint_5_flo: limit lower=-3.1416 upper=3.1416 effort=10000 velocity=6.2832 -> lower=-3.1416 upper=3.1416 effort=10 velocity=6.2832
- joint joint_6_flo: limit lower=-6.2832 upper=6.2832 effort=10000 velocity=6.2832 -> lower=-6.2832 upper=6.2832 effort=10 velocity=6.2832
- joint joint_turn_table: limit effort=10000 velocity=6.1832 -> effort=10 velocity=6.1832
